Commit message: 1st Commit

File: mockbotc1_description/urdf/common_properties.urdf.xacro (robot description, xacro)
@@ -1,4 +1,4 @@
 <?xml version="1.0" ?>
-<!-- Based on Turtlebot & Turtlebot4 - Various useful macros called in mtbc1.urdf.xacro -->
+<!-- Based on Turtlebot & Turtlebot4 - Various useful macros called in mockbotc1.urdf.xacro -->
 <robot name="xacro_properties" xmlns:xacro="http://ros.org/wiki/xacro">
   <xacro:macro name="inertial_cuboid_with_pose" params="mass x y z *origin">

File: mockbotc1_description/urdf/mockbotc1_sensors.urdf.xacro (robot description, xacro)
@@ -1,10 +1,10 @@
 <?xml version="1.0" ?>
 <robot xmlns:xacro="http://ros.org/wiki/xacro">
-  <!-- mtbc1 Sensor Models based on Turtlebot4 -->
-  <xacro:include filename="$(find mtbc1_description)/urdf/sensors/imu.urdf.xacro" />
-  <xacro:include filename="$(find mtbc1_description)/urdf/sensors/oakd.urdf.xacro" />
-  <xacro:include filename="$(find mtbc1_description)/urdf/sensors/camera_bracket.urdf.xacro" />
-  <xacro:include filename="$(find mtbc1_description)/urdf/sensors/rplidar.urdf.xacro" />
-  <xacro:include filename="$(find mtbc1_description)/urdf/sensors/sensors_shelf.urdf.xacro" />
+  <!-- mockbotc1 Sensor Models based on Turtlebot4 -->
+  <xacro:include filename="$(find mockbotc1_description)/urdf/sensors/imu.urdf.xacro" />
+  <xacro:include filename="$(find mockbotc1_description)/urdf/sensors/oakd.urdf.xacro" />
+  <xacro:include filename="$(find mockbotc1_description)/urdf/sensors/camera_bracket.urdf.xacro" />
+  <xacro:include filename="$(find mockbotc1_description)/urdf/sensors/rplidar.urdf.xacro" />
+  <xacro:include filename="$(find mockbotc1_description)/urdf/sensors/sensors_shelf.urdf.xacro" />
   <!-- TB4 sensors definitions from turtlebot4.urdf.xacro,revised for turtlebot createC1 with gazebo parameters deleted-->
   <!-- Mechanical properties -->
@@ -19,5 +19,5 @@
   <xacro:property name="oakd_lite_z_offset"             value="${9.25385*cm2m}"/>
   <xacro:property name="imu_z_offset" value="${14.1*cm2m}" />
-  <!-- For Turtlebot4 sensor xacros , MUST match xacro mtbc1.urdf.xacro xacro:name-->
+  <!-- For Turtlebot4 sensor xacros , MUST match xacro mockbotc1.urdf.xacro xacro:name-->
   <xacro:rplidar name="rplidar" parent_link="base_link">
     <origin xyz="${rplidar_x_offset} ${rplidar_y_offset} ${rplidar_z_offset + shelf_zoff}"

File: mockbotc1_description/urdf/sensors/camera_bracket.urdf.xacro (robot description, xacro)
@@ -1,6 +1,6 @@
 <?xml version="1.0"?>
-<!-- Based on Turtlebot4 and called by mtbc1_sensors.urdf.xacro -->
+<!-- Based on Turtlebot4 and called by mockbotc1_sensors.urdf.xacro -->
 <robot xmlns:xacro="http://ros.org/wiki/xacro">
-<xacro:include filename="$(find mtbc1_description)/urdf/common_properties.urdf.xacro"/>
+<xacro:include filename="$(find mockbotc1_description)/urdf/common_properties.urdf.xacro"/>
 <xacro:macro name="camera_bracket" params="name parent_link:=shell_link *origin">
   <xacro:property name="mass" value="0.033"/>
@@ -15,5 +15,5 @@
     <visual>
       <geometry>
-       <mesh filename="package://mtbc1_description/meshes/camera_bracket.dae" scale="1 1 1" />
+       <mesh filename="package://mockbotc1_description/meshes/camera_bracket.dae" scale="1 1 1" />
       </geometry>
     </visual>

File: mockbotc1_description/urdf/sensors/imu.urdf.xacro (robot description, xacro)
@@ -1,4 +1,4 @@
 <?xml version="1.0"?>
-<!-- Uses Oak-D-Lite urdf and called by mtbc1_sensors.urdf.xacro -->
+<!-- Uses Oak-D-Lite urdf and called by mockbotc1_sensors.urdf.xacro -->
 <robot xmlns:xacro="http://ros.org/wiki/xacro">
   <xacro:macro name="imu">

File: mockbotc1_description/urdf/sensors/oakd.urdf.xacro (robot description, xacro)
@@ -24,5 +24,5 @@
     <visual>
       <geometry>
-        <mesh filename="package://mtbc1_description/meshes/${name}_${model}.dae" scale="1 1 1" />
+        <mesh filename="package://mockbotc1_description/meshes/${name}_${model}.dae" scale="1 1 1" />
       </geometry>
     </visual>

File: mockbotc1_description/urdf/sensors/rplidar.urdf.xacro (robot description, xacro)
@@ -3,5 +3,5 @@
 <robot xmlns:xacro="http://ros.org/wiki/xacro">
 <xacro:macro name="rplidar" params="name parent_link *origin">
-  <xacro:include filename="$(find mtbc1_description)/urdf/common_properties.urdf.xacro"/>
+  <xacro:include filename="$(find mockbotc1_description)/urdf/common_properties.urdf.xacro"/>
   <xacro:property name="mass"       value="0.17"/>
   <xacro:property name="length_x"   value="${7.1*cm2m}" />
@@ -19,5 +19,5 @@
     <visual>
       <geometry>
-        <mesh filename="package://mtbc1_description/meshes/rplidar.dae" scale="1 1 1" />
+        <mesh filename="package://mockbotc1_description/meshes/rplidar.dae" scale="1 1 1" />
       </geometry>
     </visual>

File: mockbotc1_description/urdf/sensors/sensors_shelf.urdf.xacro (robot description, xacro)
@@ -1,4 +1,4 @@
 <?xml version="1.0"?>
-  <!-- Added to mtbc1.description and called by mtbc1_sensors.urdf.xacro -->
+  <!-- Added to mockbotc1.description and called by mockbotc1_sensors.urdf.xacro -->
   <!-- Based on shell_link & joint declaration in /standard/turtlebot4_urdf.xacro -->
 <robot name="Sensors" xmlns:xacro="http://ros.org/wiki/xacro">

File: mockbotc1_description/urdf/stacks/circlesc1.urdf.xacro (robot description, xacro)
@@ -1,5 +1,5 @@
 <?xml version="1.0"?>
 <!-- Based on Turtlebot Create revised for Mock TurtleBot Create1 -->
-<robot name="mtbc1_hardware" xmlns:xacro="http://ros.org/wiki/xacro">
+<robot name="mockbotc1_hardware" xmlns:xacro="http://ros.org/wiki/xacro">
   <xacro:macro name="stack_circles" params="parent_link">
     <joint name="plate_0_joint" type="fixed">
@@ -19,5 +19,5 @@
         <origin xyz=" 0 0 0 " rpy="0 0 0" />
         <geometry>
-          <mesh filename="package://mtbc1_description/meshes/stacks/circles/plate_0_logo.dae"/>
+          <mesh filename="package://mockbotc1_description/meshes/stacks/circles/plate_0_logo.dae"/>
         </geometry>
       </visual>
@@ -45,5 +45,5 @@
         <origin xyz=" 0 0 0 " rpy="0 0 0" />
         <geometry>
-          <mesh filename="package://mtbc1_description/meshes/stacks/circles/plate_1_logo.dae"/>
+          <mesh filename="package://mockbotc1_description/meshes/stacks/circles/plate_1_logo.dae"/>
         </geometry>
       </visual>
@@ -71,5 +71,5 @@
         <origin xyz=" 0 0 0 " rpy="0 0 0" />
         <geometry>
-          <mesh filename="package://mtbc1_description/meshes/stacks/circles/plate_2_logo.dae"/>
+          <mesh filename="package://mockbotc1_description/meshes/stacks/circles/plate_2_logo.dae"/>
         </geometry>
       </visual>
