Commit message: squash commits

File: mockbotc1_description/urdf/common_properties.urdf.xacro (robot description, xacro)
@@ -1,5 +1,9 @@
 <?xml version="1.0" ?>
-<!-- Based on Turtlebot & Turtlebot4 - Various useful macros called in mockbotc1.urdf.xacro -->
+<!-- Based on Turtlebot & slgrobotics - Various useful macros called in mockbotc1.urdf.xacro -->
 <robot name="xacro_properties" xmlns:xacro="http://ros.org/wiki/xacro">
+  <xacro:property name="PI" value="3.1415926535897931" />
+  <!-- Josh Newans articubot_one -->
+  <!-- Specify some standard inertial calculations https://en.wikipedia.org/wiki/List_of_moments_of_inertia -->
+  <!-- These make use of xacro's mathematical functionality -->
   <xacro:macro name="inertial_cuboid_with_pose" params="mass x y z *origin">
     <inertial>
@@ -11,5 +15,5 @@
     </inertial>
   </xacro:macro>
-  <xacro:macro name="inertial_cuboid" params="mass x y z">
+  <xacro:macro name="inertial_cuboid" params="mass x y z *origin">
     <xacro:inertial_cuboid_with_pose mass="${mass}" x="${x}" y="${y}" z="${z}">
       <origin xyz="0 0 0" />
@@ -25,15 +29,38 @@
     </inertial>
   </xacro:macro>
-  <xacro:macro name="inertial_cylinder" params="mass radius length">
-    <xacro:inertial_cylinder_with_pose mass="${mass}" radius="${radius}" length="${length}">
-      <origin xyz="0 0 0" />
-    </xacro:inertial_cylinder_with_pose>
+  <xacro:macro name="inertial_sphere" params="mass radius *origin">
+      <inertial>
+          <xacro:insert_block name="origin"/>
+          <mass value="${mass}" />
+          <inertia ixx="${(2/5) * mass * (radius*radius)}" ixy="0.0" ixz="0.0"
+                   iyy="${(2/5) * mass * (radius*radius)}" iyz="0.0"
+                   izz="${(2/5) * mass * (radius*radius)}" />
+      </inertial>
   </xacro:macro>
-  <xacro:macro name="inertial_sphere" params="mass radius">
+  <xacro:macro name="inertial_box" params="mass x y z *origin">
     <inertial>
+        <xacro:insert_block name="origin"/>
+        <mass value="${mass}" />
+        <inertia ixx="${(1/12) * mass * (y*y+z*z)}" ixy="0.0" ixz="0.0"
+                 iyy="${(1/12) * mass * (x*x+z*z)}" iyz="0.0"
+                 izz="${(1/12) * mass * (x*x+y*y)}" />
+    </inertial>
+  </xacro:macro>
+  <xacro:macro name="inertial_cylinder" params="mass length radius *origin">
+    <inertial>
+        <xacro:insert_block name="origin"/>
+        <mass value="${mass}" />
+        <inertia ixx="${(1/12) * mass * (3*radius*radius + length*length)}" ixy="0.0" ixz="0.0"
+                 iyy="${(1/12) * mass * (3*radius*radius + length*length)}" iyz="0.0"
+                 izz="${(1/2) * mass * (radius*radius)}" />
+    </inertial>
+   </xacro:macro>
+  <xacro:macro name="inertial_sphere" params="mass radius *origin">
+    <inertial>
+      <xacro:insert_block name="origin"/>
       <mass value="${mass}" />
-      <inertia ixx="${(2/5) * mass * radius * radius}" ixy="0.0" ixz="0.0"
-	             iyy="${(2/5) * mass * radius * radius}" iyz="0.0"
-	             izz="${(2/5) * mass * radius * radius}" />
+      <inertia ixx="${(2/5) * mass * (radius*radius)}" ixy="0.0" ixz="0.0"
+               iyy="${(2/5) * mass * (radius*radius)}" iyz="0.0"
+               izz="${(2/5) * mass * (radius*radius)}" />
     </inertial>
   </xacro:macro>
@@ -47,4 +74,23 @@
   <xacro:property name="deg2rad" value="${pi/180.0}"/>
 <!-- Material colors -->
+<!-- From create_robot -->
+  <material name="black">
+    <color rgba="0 0 0 1"/>
+  </material>
+  <material name="white">
+    <color rgba="1 1 1 1"/>
+  </material>
+  <material name="red">
+        <color rgba="1 0 0 1"/>
+  </material>
+  <material name="grey">
+    <color rgba="0.5 0.5 0.5 1"/>
+  </material>
+  <material name="green">
+    <color rgba="0.0 1.0 0.0 1.0"/>
+  </material>
+  <material name="shadow_grey">
+        <color rgba="0.3 0.3 0.3 0.5"/>
+  </material>
 <!-- From Turtlebot -->
     <xacro:property name="material_white">

File: mockbotc1_description/urdf/create_base.urdf.xacro (robot description, xacro)
@@ -1,242 +1,154 @@
 <?xml version="1.0" ?>
-<robot xmlns:xacro="http://ros.org/wiki/xacro">
-  <xacro:property name="PI" value="3.1415926535897931" />
-  <material name="black">
-    <color rgba="0 0 0 1"/>
-  </material>
-  <material name="white">
-    <color rgba="1 1 1 1"/>
-  </material>
-  <material name="grey">
-    <color rgba="0.5 0.5 0.5 1"/>
-  </material>
-  <material name="green">
-    <color rgba="0.0 1.0 0.0 1.0"/>
-  </material>
+<!-- Based on Josh Newans Articubot-One and slgrobotics -->
+<robot name="create_1" xmlns:xacro="http://ros.org/wiki/xacro">
+  <!-- mesh varient -->
+  <!-- <xacro:macro name="create_base" params="wheel_separation base_diameter base_length wheel_width wheel_radius wheel_zoffset mass_kg *mesh">
+  -->
+  <!-- Geometry Cylinder varient -->
+  <xacro:macro name="create_base" params="wheel_separation base_diameter base_length wheel_radius wheel_width wheel_zoffset mass_kg ">
+  <xacro:property name="footprint_to_base_zoffset" value="${(base_length/2+wheel_radius-wheel_zoffset)}"/>
   <xacro:macro name="create_wheel" params="prefix y_offset wheel_radius wheel_width">
     <link name="${prefix}_wheel_link">
-    <inertial>
-      <origin xyz="0 0 0" />
-      <mass value="0.01" />
-      <inertia ixx="0.001" ixy="0.0" ixz="0.0" iyy="0.001" iyz="0.0" izz="0.001" />
-    </inertial>
-    <visual>
-      <origin xyz="0 0 0" rpy="0 ${PI/2} ${PI/2}" />
-      <geometry>
-        <cylinder radius="${wheel_radius}" length="${wheel_width}" />
-      </geometry>
-      <material name="grey"/>
-    </visual>
-    <collision>
-      <origin xyz="0 0 0" rpy="0 ${PI/2} ${PI/2}" />
-      <geometry>
-        <cylinder radius="${wheel_radius}" length="${wheel_width}" />
-      </geometry>
-    </collision>
+      <visual>
+        <origin xyz="0 0 0" rpy="0 ${pi/2} ${pi/2}"/>
+        <geometry>
+          <cylinder radius="${wheel_radius}" length="${wheel_width}"/>
+        </geometry>
+        <material name="grey"/>
+      </visual>
+      <collision>
+        <origin xyz="0 0 0" rpy="0 ${pi/2} ${pi/2}"/>
+        <geometry>
+          <cylinder radius="${wheel_radius}" length="${wheel_width}"/>
+        </geometry>
+      </collision>
+      <xacro:inertial_cylinder mass="0.01" length="${wheel_width}" radius="${wheel_radius}">
+        <origin xyz="0 0 0" rpy="0 0 0"/>
+      </xacro:inertial_cylinder>
     </link>
-   <joint name="${prefix}_wheel_joint" type="continuous">
-      <!-- <origin xyz="0 ${y_offset} 0.015" rpy="0 0 0" /> -->
-      <origin xyz="0 ${y_offset} ${-(footprint_to_base_zoffset-wheel_radius-wheel_zoffset)}" rpy="0 0 0" />
-      <parent link="base_link" />
-      <child link="${prefix}_wheel_link" />
-      <axis xyz="0 1 0" />
+    <!-- joint name="${prefix}_wheel_joint" type="fixed" -->
+    <joint name="wheel_${prefix}_joint" type="continuous">
+      <origin xyz="0 ${y_offset} ${-wheel_radius}" rpy="0 0 0"/>
+      <parent link="chassis_link"/>
+      <child link="${prefix}_wheel_link"/>
+      <axis xyz="0 1 0"/>
     </joint>
   </xacro:macro>
-  <!-- mesh varient -->
-  <xacro:macro name="create_base" params="diffdrive_update_rate:=40 wheel_separation wheel_radius:=0.036 wheel_width:=0.024 wheel_zoffset:=0.005 wheel_torque:=1.0 wheel_accel:=1.8 mass_kg:=3.5 base_diameter base_length *mesh">
-  <!-- Geometry Cylinder varient -->
-  <!-- <xacro:macro name="create_base" params="diffdrive_update_rate:=40 wheel_separation wheel_radius:=0.036 wheel_width:=0.024 wheel_zoffset:=0.005 wheel_torque:=1.0 wheel_accel:=1.8 mass_kg:=3.5 base_diameter base_length"> -->
-  <xacro:property name="footprint_to_base_zoffset" value="${(base_length/2+wheel_radius-wheel_zoffset)}"/>
-  <!--<xacro:include filename="$(find create_description)/urdf/create_base_gazebo.urdf.xacro" /> -->
-    <!-- Robot Footprint -->
-    <!-- Follows syntax of Nav2 Sambot -->
+    <!-- The coordinate frame called base_link is rigidly attached to the robot root body. -->
+    <link name="base_link">
+      <visual name="baselink_visual">
+          <origin xyz="0 0 0"/>
+          <geometry>
+              <sphere radius="0.01"/>
+          </geometry>
+          <material name="black"/>
+      </visual>
+    </link>
+    <!-- Define the center of the main robot chassis projected on the ground -->
     <link name="base_footprint">
-     <visual>
-       <origin xyz="0 0 0" rpy="0 0 0" />
-       <geometry>
-         <box size="0.001 0.001 0.001" />
-       </geometry>
-       <material name="green" />
-     </visual>
-     <collision>
-       <origin xyz="0.0 0.0 ${-(0.045)}" rpy="0 0 0" />
-       <geometry>
-         <box size="0.001 0.001 0.001" />
-       </geometry>
+      <visual name="footprint_visual">
+          <origin xyz="0 0 0"/>
+          <geometry>
+              <cylinder radius="${base_diameter/2 + 0.01}" length="0.003"/>
+          </geometry>
+          <material name="shadow_grey"/>
+      </visual>
+    </link>
+    <!-- The base footprint of the robot is located underneath the chassis -->
+    <joint name="base_footprint_joint" type="fixed">
+      <parent link="base_link"/>
+      <child link="base_footprint" />
+      <origin xyz="0 0 -${wheel_radius}" rpy="0 0 0"/>
+    </joint>
+    <joint name="chassis_joint" type="fixed">
+      <parent link="base_link"/>
+      <child link="chassis_link"/>
+      <origin xyz="0 0 ${wheel_radius}"/>
+    </joint>
+    <!-- CHASSIS LINK -->
+    <link name="chassis_link">
+      <visual name="chassis_rviz_visual">
+        <origin xyz=" 0 0 -0.015" rpy="0 0 0"/>
+        <geometry>
+          <!-- Mesh varient -->
+          <!-- <xacro:insert_block name="mesh"/> -->
+          <!-- Geometry Varient-->
+          <cylinder length="${base_length}" radius="${base_diameter/2}"/>
+        </geometry>
+        <material name="white"/>
+      </visual>
+      <collision>
+        <origin xyz="0.0 0.0 0" rpy="0 0 0"/>
+        <geometry>
+          <cylinder length="0.0611632" radius="${base_diameter/2}"/>
+        </geometry>
       </collision>
-    </link>
-    <!-- Revised base_link & base_footprint -->
-    <joint name="base_footprint_joint" type="fixed">
-      <!--<origin xyz="0.0 0.0 ${-(0.045)}" rpy="0 0 0" />-->
-      <origin xyz="0.0 0.0 ${-(footprint_to_base_zoffset)}" rpy="0 0 0" />
-      <parent link="base_link" />
-      <child link="base_footprint" />
-    </joint>
-    <!-- Robot Link -->
-    <!-- Revised origin to 0 0 0 -->
-    <link name="base_link">
-     <inertial>
-       <mass value="2" />
-       <origin xyz="0.0 0.0 0.0" />
-       <inertia ixx="0.01" ixy="0.0" ixz="0.0" iyy="0.01" iyz="0.0" izz="0.5" />
-     </inertial>
-     <visual>
-      <origin xyz=" 0 0 0" rpy="0 0 0" />
-      <geometry>
-        <!-- Mesh varient -->
-        <xacro:insert_block name="mesh" />
-        <!-- Geometry Cylinder varient -->
-        <!-- <cylinder radius="${base_diameter/2}" length="${base_length}"/> -->
-      </geometry>
-      <material name="white"/>
-     </visual>
-     <collision>
-      <origin xyz="0.0 0.0 0.0" rpy="0 0 0" />
-      <geometry>
-        <cylinder length="0.0611632" radius="0.16495" />
-      </geometry>
-     </collision>
+      <xacro:inertial_cylinder mass="${mass_kg}" length="${base_length}" radius="${base_diameter/2}">
+        <!-- cheat: origin moved forward a bit, so that center mass is forward of the wheels axis -->
+        <origin xyz="0.03 0 0" rpy="0 0 0"/>
+      </xacro:inertial_cylinder>
     </link>
     <link name="wall_sensor_link">
-    <inertial>
-      <mass value="0.01" />
-      <origin xyz="0 0 0" />
-      <inertia ixx="0.001" ixy="0.0" ixz="0.0" iyy="0.001" iyz="0.0" izz="0.001" />
-    </inertial>
     </link>
     <link name="left_cliff_sensor_link">
-    <inertial>
-      <mass value="0.01" />
-      <origin xyz="0 0 0" />
-      <inertia ixx="0.001" ixy="0.0" ixz="0.0" iyy="0.001" iyz="0.0" izz="0.001" />
-    </inertial>
     </link>
     <link name="right_cliff_sensor_link">
-    <inertial>
-      <mass value="0.01" />
-      <origin xyz="0 0 0" />
-      <inertia ixx="0.001" ixy="0.0" ixz="0.0" iyy="0.001" iyz="0.0" izz="0.001" />
-    </inertial>
     </link>
     <link name="leftfront_cliff_sensor_link">
-    <inertial>
-      <mass value="0.01" />
-      <origin xyz="0 0 0" />
-      <inertia ixx="1.0" ixy="0.0" ixz="0.0" iyy="0.01" iyz="0.0" izz="0.01" />
-    </inertial>
     </link>
     <link name="rightfront_cliff_sensor_link">
-    <inertial>
-      <mass value="0.01" />
-      <origin xyz="0 0 0" />
-      <inertia ixx="0.001" ixy="0.0" ixz="0.0" iyy="0.001" iyz="0.0" izz="0.001" />
-    </inertial>
     </link>
     <joint name="base_wall_sensor_joint" type="fixed">
-      <origin xyz="0.09 -0.120 0.042" rpy="0 0 -1.0" />
-      <parent link="base_link" />
-      <child link="wall_sensor_link" />
+      <origin xyz="0.09 -0.120 0.042" rpy="0 0 -1.0"/>
+      <parent link="chassis_link"/>
+      <child link="wall_sensor_link"/>
     </joint>
     <joint name="base_left_cliff_sensor_joint" type="fixed">
-      <origin xyz="0.07 0.14 0.01" rpy="0 ${PI/2} 0" />
-      <parent link="base_link" />
-      <child link="left_cliff_sensor_link" />
+      <origin xyz="0.07 0.14 0.01" rpy="0 ${pi/2} 0"/>
+      <parent link="chassis_link"/>
+      <child link="left_cliff_sensor_link"/>
     </joint>
     <joint name="base_right_cliff_sensor_joint" type="fixed">
-      <origin xyz="0.07 -0.14 0.01" rpy="0 ${PI/2} 0" />
-      <parent link="base_link" />
-      <child link="right_cliff_sensor_link" />
+      <origin xyz="0.07 -0.14 0.01" rpy="0 ${pi/2} 0"/>
+      <parent link="chassis_link"/>
+      <child link="right_cliff_sensor_link"/>
     </joint>
     <joint name="base_leftfront_cliff_sensor_joint" type="fixed">
-      <origin xyz="0.15 0.04 0.01" rpy="0 ${PI/2} 0" />
-      <parent link="base_link" />
-      <child link="leftfront_cliff_sensor_link" />
+      <origin xyz="0.15 0.04 0.01" rpy="0 ${pi/2} 0"/>
+      <parent link="chassis_link"/>
+      <child link="leftfront_cliff_sensor_link"/>
     </joint>
     <joint name="base_rightfront_cliff_sensor_joint" type="fixed">
-      <origin xyz="0.15 -0.04 0.01" rpy="0 ${PI/2} 0" />
-      <parent link="base_link" />
-      <child link="rightfront_cliff_sensor_link" />
+      <origin xyz="0.15 -0.04 0.01" rpy="0 ${pi/2} 0"/>
+      <parent link="chassis_link"/>
+      <child link="rightfront_cliff_sensor_link"/>
     </joint>
     <xacro:create_wheel prefix="left" y_offset="${wheel_separation / 2}" wheel_radius="${wheel_radius}" wheel_width="${wheel_width}"/>
     <xacro:create_wheel prefix="right" y_offset="${wheel_separation / -2}" wheel_radius="${wheel_radius}" wheel_width="${wheel_width}"/>
-    <link name="rear_wheel_link">
-    <inertial>
-      <origin xyz="0 0 0"/>
-      <mass value="0.001" />
-      <inertia ixx="0.0001" ixy="0.0" ixz="0.0"
-        iyy="0.0001" iyz="0.0" izz="0.0001" />
-    </inertial>
-    <visual>
-      <origin xyz="0 0 0" rpy="0 ${PI/2} ${PI/2}"/>
-      <geometry>
-        <sphere radius="0.015" />
-      </geometry>
-      <material name="grey"/>
-    </visual>
-    <collision>
-      <origin xyz="0 0 0" rpy="0 ${PI/2} ${PI/2}" />
-      <geometry>
-        <sphere radius="0.015" />
-      </geometry>
-    </collision>
-    </link>
-    <joint name="rear_castor_joint" type="fixed">
-      <!--<origin xyz="-0.13 0 0.0" rpy="0 0 0"/>-->
-      <origin xyz="-0.13 0 ${-(footprint_to_base_zoffset-0.015)}" rpy="0 0 0"/>
-      <parent link="base_link"/>
-      <child link="rear_wheel_link"/>
-      <axis xyz="0 1 0"/>
-    </joint>
-    <link name="front_wheel_link">
-    <inertial>
-      <origin xyz="0 0 0" />
-      <mass value="0.01" />
-      <inertia ixx="0.001" ixy="0.0" ixz="0.0" iyy="0.001" iyz="0.0" izz="0.001" />
-    </inertial>
-    <visual>
-      <origin xyz="0 0 0" rpy="0 ${PI/2} ${PI/2}" />
-      <geometry>
-        <sphere radius="0.018" />
-      </geometry>
-      <material name="grey"/>
-    </visual>
-    <collision>
-      <origin xyz="0 0 0" rpy="0 ${PI/2} ${PI/2}" />
-      <geometry>
-        <sphere radius="0.018" />
-      </geometry>
-    </collision>
+    <link name="front_castor_link">
+      <visual>
+        <origin xyz="0 0 0" rpy="0 ${pi/2} ${pi/2}"/>
+        <geometry>
+          <sphere radius="0.018"/>
+        </geometry>
+        <material name="grey"/>
+      </visual>
+      <collision>
+        <origin xyz="0 0 0" rpy="0 ${pi/2} ${pi/2}"/>
+        <geometry>
+          <sphere radius="0.018"/>
+        </geometry>
+      </collision>
+      <xacro:inertial_sphere mass="0.01" radius="0.018">
+        <origin xyz="0 0 0" rpy="0 0 0"/>
+      </xacro:inertial_sphere>
     </link>
     <!-- fixed because there's no transmission -->
     <joint name="front_castor_joint" type="fixed">
-      <!-- <origin xyz="0.13 0 0.0" rpy="0 0 0" /> -->
-      <origin xyz="0.13 0 ${-(footprint_to_base_zoffset-0.018)}" rpy="0 0 0" />
-      <parent link="base_link" />
-      <child link="front_wheel_link" />
-      <axis xyz="0 1 0" />
+      <origin xyz="0.13 0 -0.048" rpy="0 0 0"/>
+      <parent link="chassis_link"/>
+      <child link="front_castor_link"/>
+      <axis xyz="0 1 0"/>
     </joint>
-    <!-- Gyro Sensor -->
-    <!-- Disable Gyro Sensors
-    <joint name="gyro_joint" type="fixed">
-      <axis xyz="0 1 0" />
-      <origin xyz="0 0 0.04" rpy="0 0 0" />
-      <parent link="base_link" />
-      <child link="gyro_link" />
-    </joint>
-    <link name="gyro_link">
-    <inertial>
-      <mass value="0.001" />
-      <origin xyz="0 0 0" rpy="0 0 0" />
-      <inertia ixx="0.0001" ixy="0" ixz="0" iyy="0.000001" iyz="0" izz="0.0001" />
-    </inertial>
-    </link>
-    -->
-    <!-- Simulation Sensors -->
-    <!-- Disable Simulation
-    <xacro:sim_create_base/>
-    <xacro:sim_create_wall_sensor/>
-    <xacro:sim_create_cliff_sensors/>
-    <xacro:sim_imu/>
-     -->
   </xacro:macro>
 </robot>

File: mockbotc1_description/urdf/mockbotc1.urdf.xacro (robot description, xacro)
@@ -8,11 +8,9 @@
   <!-- <xacro:include filename="$(find mockbotc1_description)/urdf/sensors/sensors_shelf.urdf.xacro" /> -->
   <!-- <xacro:include filename="$(find mockbotc1_description)/urdf/mockbotc1_sensors.urdf.xacro"/> -->
-  <!-- <xacro:include filename="$(find mockbotc1_description)/urdf/stacks/circlesc1.urdf.xacro"/> -->
-  <!-- <xacro:create_base wheel_separation="0.26" base_diameter="0.3302"> -->
-   <xacro:create_base wheel_separation="0.26" base_diameter="${33.02*cm2m}" base_length="${6.11632*cm2m}"/>
-      <mesh filename="package://mockbotc1_description/meshes/create_1.dae" />
-  <!-- </xacro:create_base> -->
-  <!-- TB circles xacros -->
+  <xacro:include filename="$(find mockbotc1_description)/urdf/stacks/circlesc1.urdf.xacro"/>
+  <xacro:include filename="create_1.urdf.xacro"/>
+     <!-- TB circles xacros -->
   <!-- <create/> -->
   <!-- <xacro:stack_circles parent_link="base_link"/> -->
+  <xacro:stack_circles parent_link="base_link"/>
 </robot>

File: mockbotc1_description/urdf/smarty_description.urdf (robot description, URDF)
Before this commit: robot MockBOT, 14 links, 13 joints
Links:
- removed link lidar_link
- added link laser; collision cylinder length=0.05 radius=0.0375; visual cylinder length=0.025 radius=0.0375
Joints:
- joint lidar_joint: child lidar_link -> laser

File: mockbotc1_description/urdf/stacks/circlesc1.urdf.xacro (robot description, xacro)
@@ -2,5 +2,14 @@
 <!-- Based on Turtlebot Create revised for Mock TurtleBot Create1 -->
 <robot name="mockbotc1_hardware" xmlns:xacro="http://ros.org/wiki/xacro">
-  <xacro:macro name="stack_circles" params="parent_link">
+  <!-- Define Circles constants -->
+  <xacro:property name="plate_diameter" value="${31.5*cm2m}"/>
+  <xacro:property name="plate_length" value="${6*cm2m}"/>
+  <xacro:property name="standoff_length" value="${27.6*cm2m}"/>
+  <xacro:property name="standoff_diameter" value="${0.6*cm2m}"/>
+  <xacro:property name="standoff_rear_xoffset" value="${11.9*cm2m}"/>
+  <xacro:property name="standoff_front_xoffset" value="${5.0*cm2m}"/>
+  <xacro:property name="standoff_yoffset" value="${13.1*cm2m}"/>
+  <xacro:property name="standoff_zoffset" value="$(16.92*cm2m}"/>
+    <xacro:macro name="stack_circles" params="parent_link">
     <joint name="plate_0_joint" type="fixed">
       <origin xyz="-0.04334 0  0.06775704" rpy="0 0 0" />
@@ -19,6 +28,8 @@
         <origin xyz=" 0 0 0 " rpy="0 0 0" />
         <geometry>
-          <mesh filename="package://mockbotc1_description/meshes/stacks/circles/plate_0_logo.dae"/>
+        <!-- <mesh filename="package://mockbotc1_description/meshes/stacks/circles/plate_0_logo.dae"/>  -->
+        <cylindar length="${plate_length}" radius="${plate_diameter/2}"/>
         </geometry>
+        <material name="white"/>
       </visual>
       <collision>
@@ -45,6 +56,8 @@
         <origin xyz=" 0 0 0 " rpy="0 0 0" />
         <geometry>
-          <mesh filename="package://mockbotc1_description/meshes/stacks/circles/plate_1_logo.dae"/>
+          <!-- <mesh filename="package://mockbotc1_description/meshes/stacks/circles/plate_1_logo.dae"/> -->
+          <cylindar length="${plate_length}" radius="${plate_diameter/2}"/>
         </geometry>
+        <material name="white"\>
       </visual>
       <collision>
@@ -71,6 +84,8 @@
         <origin xyz=" 0 0 0 " rpy="0 0 0" />
         <geometry>
-          <mesh filename="package://mockbotc1_description/meshes/stacks/circles/plate_2_logo.dae"/>
+          <!-- <mesh filename="package://mockbotc1_description/meshes/stacks/circles/plate_2_logo.dae"/> -->
+          <cylindar plate_length="${plate_length}" plate_radius="${plate_diameter/2}"/>
         </geometry>
+        <material name="white"\>
       </visual>
       <collision>
